Commit message: task2

File: tasks/week2-4 飞控组/week2/ros_project/src/little_car/urdf/little_car.urdf (robot description, URDF)
Before this commit: robot little_car, 5 links, 4 joints
Links:
- link base_link: mass None -> 10; geometry collision box size=0.21 0.3 0.11; visual box size=0.3 0.2 0.1
- link wheel_1: mass None -> 10; geometry collision box size=0.21 0.3 0.11; visual cylinder length=0.05 radius=0.05
- link wheel_2: mass None -> 10; geometry collision box size=0.21 0.3 0.11; visual cylinder length=0.05 radius=0.05
- link wheel_3: mass None -> 10; geometry collision box size=0.21 0.3 0.11; visual cylinder length=0.05 radius=0.05
- link wheel_4: mass None -> 10; geometry collision box size=0.21 0.3 0.11; visual cylinder length=0.05 radius=0.05
Joints:
- removed joint base_to_wheel_1
- removed joint base_to_wheel_2
- removed joint base_to_wheel_3
- removed joint base_to_wheel_4
- added joint base_to_wheel1: type continuous, parent base_link, child wheel_1
- added joint base_to_wheel2: type continuous, parent base_link, child wheel_2
- added joint base_to_wheel3: type continuous, parent base_link, child wheel_3
- added joint base_to_wheel4: type continuous, parent base_link, child wheel_4
